File: pcb/sdcard-adapter.kicad_sch (KiCad schematic)
At the start: 11 parts, among them J1 SDCARD, J2 Micro_SD_Card_Det1, Q1 BSS138, Q2 BSS138, Q3 BSS138, Q4 BSS138, U1 AMS1117-3.3

Commit message: Adding step files
Parts:
- J1: footprint components:sdcard-socket -> Connector_PinHeader_2.54mm:PinHeader_1x06_P2.54mm_Vertical
- J2: footprint components:CONN9_MSD-1_CUD -> components:sdcard-socket
Changed lines of the file:
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@@
 (kicad_sch
-	(version 20231120)
+	(version 20250114)
 	(generator "eeschema")
-	(generator_version "8.0")
+	(generator_version "9.0")
 	(paper "A5")
 	(title_block
@@
 		(rev "rev0")
 	)
+	(text "SDCARD slot"
+		(exclude_from_sim no)
+		(at 152.908 18.034 0)
+		(effects
+			(font
+				(size 1.27 1.27)
+			)
+		)
+	)
+	(text "SD CARD"
+		(exclude_from_sim no)
+		(at 176.784 70.866 0)
+		(effects
+			(font
+				(size 1.27 1.27)
+			)
+			(justify left bottom)
+		)
+	)
+	(text "5v <-> 3v3 bridges"
+		(exclude_from_sim no)
+		(at 50.038 20.066 0)
+		(effects
+			(font
+				(size 1.27 1.27)
+			)
+		)
+	)
+	(text "Voltage regulator"
+		(exclude_from_sim no)
+		(at 168.656 64.008 0)
+		(effects
+			(font
+				(size 1.27 1.27)
+			)
+		)
+	)
+	(text "SCK"
+		(exclude_from_sim no)
+		(at 153.67 22.225 0)
+		(effects
+			(font
+				(size 1 1)
+			)
+			(justify left bottom)
+		)
+	)
 	(junction
 		(at 27.94 38.1)
@@
 		)
 	)
-	(text "SDCARD slot"
-		(exclude_from_sim no)
-		(at 152.908 18.034 0)
-		(effects
-			(font
-				(size 1.27 1.27)
-			)
-		)
-	)
-	(text "SD CARD"
-		(exclude_from_sim no)
-		(at 176.784 70.866 0)
-		(effects
-			(font
-				(size 1.27 1.27)
-			)
-			(justify left bottom)
-		)
-	)
-	(text "5v <-> 3v3 bridges"
-		(exclude_from_sim no)
-		(at 50.038 20.066 0)
-		(effects
-			(font
-				(size 1.27 1.27)
-			)
-		)
-	)
-	(text "Voltage regulator"
-		(exclude_from_sim no)
-		(at 168.656 64.008 0)
-		(effects
-			(font
-				(size 1.27 1.27)
-			)
-		)
-	)
-	(text "SCK"
-		(exclude_from_sim no)
-		(at 153.67 22.225 0)
-		(effects
-			(font
-				(size 1 1)
-			)
-			(justify left bottom)
-		)
-	)
 	(global_label "D0_LLS"
 		(shape input)
@@
 			)
 		)
-		(property "Footprint" "components:sdcard-socket"
+		(property "Footprint" "Connector_PinHeader_2.54mm:PinHeader_1x06_P2.54mm_Vertical"
 			(at 105.41 41.91 0)
 			(effects
@@
 			)
 		)
-		(property "Footprint" "components:CONN9_MSD-1_CUD"
+		(property "Footprint" "components:sdcard-socket"
 			(at 222.25 19.05 0)
 			(effects
@@
 		)
 	)
+	(embedded_fonts no)
 )
